File: 5V27VBoostUp(USBC-Tune)_V1.1/5V24VBoostUp(USBC).kicad_sch (KiCad schematic)
At the start: 12 parts, among them J2 Output, J3 USB_C_Receptacle_PowerOnly_6P, U1 MT3608

Commit message: Update V2
Parts:
- removed C2: 22u, Capacitor_SMD:C_0603_1608Metric_Pad1.08x0.95mm_HandSolder, symbol Device:C
- removed R1: 100k, Potentiometer_THT:Potentiometer_Bourns_3296W_Vertical, symbol Device:R_Variable
- added RV1: 100k, Potentiometer_THT:Potentiometer_Bourns_3296W_Vertical, symbol Device:R_Potentiometer_US
- C1, C3: footprint Capacitor_SMD:C_0603_1608Metric_Pad1.08x0.95mm_HandSolder -> Capacitor_SMD:C_1206_3216Metric_Pad1.33x1.80mm_HandSolder
- D1: Spec (none) -> 40V/3A
- J2: footprint Connector_PinHeader_2.00mm:PinHeader_1x02_P2.00mm_Vertical -> Connector_PinHeader_2.54mm:PinHeader_1x02_P2.54mm_Vertical
- J3: Spec (none) -> 5V@1.5A
- L1: footprint Inductor_SMD:L_6.3x6.3_H3 -> Inductor_SMD:L_7.3x7.3_H3.5
- R2: footprint Resistor_SMD:R_0603_1608Metric_Pad0.98x0.95mm_HandSolder -> Resistor_SMD:R_1206_3216Metric_Pad1.30x1.75mm_HandSolder
- R3, R4: value 5.1k -> 22k; footprint Resistor_SMD:R_0603_1608Metric_Pad0.98x0.95mm_HandSolder -> Resistor_SMD:R_1206_3216Metric_Pad1.30x1.75mm_HandSolder
Connections:
- net at C3.1, D1.1 (K), J2.1 (Pin_1): now also RV1.1
- net at U1.3 (FB): now also RV1.2; no longer R2.2
- new net: R2.2, RV1.3
Other:
- moved on the sheet: C1, C3, J2, R2
